File: aswitch/74AHC1G66GW_TSSOP/74AHC1G66GW_TSSOP.sch (KiCad schematic (older format))
At the start: 21 parts, among them P1 CONN_01X02, P10 CONN_01X01, P11 CONN_01X01, P12 CONN_01X01, P13 CONN_01X01, P14 CONN_01X01, P2 CONN_01X02, P3 CONN_01X01, P4 CONN_01X01, P5 CONN_01X01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

Commit message: Re-export gerbers at 0.1mm default line width, update .schs with KiField, wget wavegen ICL 8083
Parts:
- U1, U2, U3, U4: Dist [1] Part # (none) -> 771-AHC1G66GW125; Dist [1] Source (none) -> http://www2.mouser.com/ProductDetail/NXP-Semiconductors/74A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; Mfr (none) -> NXP; Mfr Part # (none) -> 74AHC1G66GW,125
