File: captouch/cypress-10/CY8CMBR2010.sch (KiCad schematic (older format))
At the start: 57 parts, among them P1 CONN_01X02, P10 CONN_01X01, P11 CONN_01X01, P12 CONN_01X01, P13 CONN_01X03, P14 CONN_01X03, P15 CONN_01X01, P16 CONN_01X01, P17 CONN_01X01, P18 CONN_01X01, P19 CONN_01X03, P2 CONN_01X02, P20 CONN_01X03, P21 CONN_01X01, P22 CONN_01X01, P23 CONN_01X01, P24 CONN_01X01, P25 CONN_01X01, P26 CONN_01X01, P27 CONN_01X01, P28 CONN_01X01, P29 CONN_01X01, P3 CONN_01X01, P30 CONN_01X01, P31 CONN_01X01, P4 CONN_01X10, P5 CONN_01X01, P6 CONN_01X01, P7 CONN_01X03, P8 CONN_01X01, P9 CONN_01X03, U1 CY8CMBR2010

Commit message: Re-export gerbers at 0.1mm default line width, update .schs with KiField, wget wavegen ICL 8083
Parts:
- U1: Dist [1] Part # (none) -> 727-8CMBR2010-24LQXI; Dist [1] Source (none) -> http://www2.mouser.com/ProductDetail/Cypress-Semiconductor/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; Mfr (none) -> Cypress; Mfr Part # (none) -> CY8CMBR2010-24LQXI
