File: captouch/cypress-2/cy8cmbr3002.sch (KiCad schematic (older format))
At the start: 12 parts, among them P1 CONN_01X02, P2 CONN_01X02, P3 CONN_01X02, U1 CY8CMBR3002

Commit message: Re-export gerbers at 0.1mm default line width, update .schs with KiField, wget wavegen ICL 8083
Parts:
- U1: Dist [1] Part # (none) -> 727-CY8CMBR3002-SX1I; Dist [1] Source (none) -> http://www2.mouser.com/ProductDetail/Cypress-Semiconductor/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; Mfr (none) -> Cypress; Mfr Part # (none) -> CY8CMBR3002-SX1I
Changed lines of the file:
@@
 U 1 1 57FC1C1A
 P 2850 2500
-F 0 "U1" H 2450 2850 50  0000 L CNN
-F 1 "CY8CMBR3002" H 2950 2850 50  0000 L CNN
-F 2 "SMD_Packages:SOIC-8-N" H 2850 1950 50  0001 C CNN
-F 3 "" H 2850 1950 50  0000 C CNN
+F 0 "U1" H 2450 2850 50 0000 L CNN
+F 1 "CY8CMBR3002" H 2950 2850 50 0000 L CNN
+F 2 "SMD_Packages:SOIC-8-N" H 2850 1950 50 0001 C CNN
+F 3 "" H 2850 1950 50 0000 C CNN
+F 4 "727-CY8CMBR3002-SX1I" H 0 0 50 0001 C CNN "Dist [1] Part #"
+F 5 "http://www2.mouser.com/ProductDetail/Cypress-Semiconductor/CY8CMBR3002-SX1I/?qs=%2fha2pyFadujUUTSzdwlWqpheTKjCuXJ8zaCioaEFuiFAA6NtFEWpDQ%3d%3d" H 0 0 50 0001 C CNN "Dist [1] Source"
+F 6 "CY8CMBR3002-SX1I" H 0 0 50 0001 C CNN "Mfr Part #"
+F 7 "Cypress" H 0 0 50 0001 C CNN "Mfr"
 	1    2850 2500
 	1    0    0    -1
@@
 U 1 1 57FC1C65
 P 3500 2800
-F 0 "C4" H 3510 2870 50  0000 L CNN
-F 1 "0.1uF" H 3510 2720 50  0000 L CNN
-F 2 "Capacitors_SMD:C_1206_HandSoldering" H 3500 2800 50  0001 C CNN
-F 3 "" H 3500 2800 50  0000 C CNN
+F 0 "C4" H 3510 2870 50 0000 L CNN
+F 1 "0.1uF" H 3510 2720 50 0000 L CNN
+F 2 "Capacitors_SMD:C_1206_HandSoldering" H 3500 2800 50 0001 C CNN
+F 3 "" H 3500 2800 50 0000 C CNN
 	1    3500 2800
 	1    0    0    -1
 $EndComp
-Wire Wire Line
-	3350 2600 3500 2600
-Wire Wire Line
-	3500 2600 3500 2700
 $Comp
 L GND #PWR01
 U 1 1 57FC1CCD
 P 2850 3000
-F 0 "#PWR01" H 2850 2750 50  0001 C CNN
-F 1 "GND" H 2850 2850 50  0000 C CNN
-F 2 "" H 2850 3000 50  0000 C CNN
-F 3 "" H 2850 3000 50  0000 C CNN
+F 0 "#PWR01" H 2850 2750 50 0001 C CNN
+F 1 "GND" H 2850 2850 50 0000 C CNN
+F 2 "" H 2850 3000 50 0000 C CNN
+F 3 "" H 2850 3000 50 0000 C CNN
 	1    2850 3000
 	1    0    0    -1
 $EndComp
-Wire Wire Line
-	2850 2900 2850 3000
-Wire Wire Line
-	2200 2950 3500 2950
-Wire Wire Line
-	3500 2950 3500 2900
-Connection ~ 2850 2950
 $Comp
 L C_Small C3
 U 1 1 57FC1E00
 P 2200 2800
-F 0 "C3" H 2210 2870 50  0000 L CNN
-F 1 "2.2nF" H 2210 2720 50  0000 L CNN
-F 2 "Capacitors_SMD:C_1206_HandSoldering" H 2200 2800 50  0001 C CNN
-F 3 "" H 2200 2800 50  0000 C CNN
-F 4 "5V X7R/NP0" H 2200 2800 60  0001 C CNN "Tolerance"
+F 0 "C3" H 2210 2870 50 0000 L CNN
+F 1 "2.2nF" H 2210 2720 50 0000 L CNN
+F 2 "Capacitors_SMD:C_1206_HandSoldering" H 2200 2800 50 0001 C CNN
+F 3 "" H 2200 2800 50 0000 C CNN
+F 4 "5V X7R/NP0" H 2200 2800 60 0001 C CNN "Tolerance"
 	1    2200 2800
 	1    0    0    -1
 $EndComp
-Wire Wire Line
-	2350 2600 2200 2600
-Wire Wire Line
-	2200 2600 2200 2700
-Wire Wire Line
-	2200 2900 2200 2950
 $Comp
 L R_Small R3
 U 1 1 57FC1ED4
 P 2100 2400
-F 0 "R3" H 2130 2420 50  0000 L CNN
-F 1 "560" H 2130 2360 50  0000 L CNN
-F 2 "Capacitors_SMD:C_1206_HandSoldering" H 2100 2400 50  0001 C CNN
-F 3 "" H 2100 2400 50  0000 C CNN
+F 0 "R3" H 2130 2420 50 0000 L CNN
+F 1 "560" H 2130 2360 50 0000 L CNN
+F 2 "Capacitors_SMD:C_1206_HandSoldering" H 2100 2400 50 0001 C CNN
+F 3 "" H 2100 2400 50 0000 C CNN
 	1    2100 2400
 	0    1    1    0
@@
 U 1 1 57FC1F2D
 P 2100 2300
-F 0 "R1" H 2130 2320 50  0000 L CNN
-F 1 "560" H 2130 2260 50  0000 L CNN
-F 2 "Capacitors_SMD:C_1206_HandSoldering" H 2100 2300 50  0001 C CNN
-F 3 "" H 2100 2300 50  0000 C CNN
+F 0 "R1" H 2130 2320 50 0000 L CNN
+F 1 "560" H 2130 2260 50 0000 L CNN
+F 2 "Capacitors_SMD:C_1206_HandSoldering" H 2100 2300 50 0001 C CNN
+F 3 "" H 2100 2300 50 0000 C CNN
 	1    2100 2300
 	0    -1   -1   0
 $EndComp
-Wire Wire Line
-	2350 2300 2200 2300
-Wire Wire Line
-	2350 2400 2200 2400
-Wire Wire Line
-	2000 2300 1850 2300
-Wire Wire Line
-	2000 2400 1850 2400
-Wire Wire Line
-	2850 2050 2850 2100
 $Comp
 L VDD #PWR02
 U 1 1 57FC225B
 P 2850 2050
-F 0 "#PWR02" H 2850 1900 50  0001 C CNN
-F 1 "VDD" H 2850 2200 50  0000 C CNN
-F 2 "" H 2850 2050 50  0000 C CNN
-F 3 "" H 2850 2050 50  0000 C CNN
+F 0 "#PWR02" H 2850 1900 50 0001 C CNN
+F 1 "VDD" H 2850 2200 50 0000 C CNN
+F 2 "" H 2850 2050 50 0000 C CNN
+F 3 "" H 2850 2050 50 0000 C CNN
 	1    2850 2050
 	1    0    0    -1
@@
 U 1 1 57FC24A7
 P 3600 2300
-F 0 "R2" H 3630 2320 50  0000 L CNN
-F 1 "10k" H 3630 2260 50  0000 L CNN
-F 2 "Capacitors_SMD:C_1206_HandSoldering" H 3600 2300 50  0001 C CNN
-F 3 "" H 3600 2300 50  0000 C CNN
+F 0 "R2" H 3630 2320 50 0000 L CNN
+F 1 "10k" H 3630 2260 50 0000 L CNN
+F 2 "Capacitors_SMD:C_1206_HandSoldering" H 3600 2300 50 0001 C CNN
+F 3 "" H 3600 2300 50 0000 C CNN
 	1    3600 2300
 	0    -1   -1   0
 $EndComp
-Wire Wire Line
-	3500 2300 3350 2300
-Wire Wire Line
-	3350 2400 3500 2400
 $Comp
 L R_Small R4
 U 1 1 57FC2567
 P 3600 2400
-F 0 "R4" H 3630 2420 50  0000 L CNN
-F 1 "10k" H 3630 2360 50  0000 L CNN
-F 2 "Capacitors_SMD:C_1206_HandSoldering" H 3600 2400 50  0001 C CNN
-F 3 "" H 3600 2400 50  0000 C CNN
+F 0 "R4" H 3630 2420 50 0000 L CNN
+F 1 "10k" H 3630 2360 50 0000 L CNN
+F 2 "Capacitors_SMD:C_1206_HandSoldering" H 3600 2400 50 0001 C CNN
+F 3 "" H 3600 2400 50 0000 C CNN
 	1    3600 2400
 	0    1    1    0
@@
 U 1 1 57FC26AD
 P 4050 2350
-F 0 "P3" H 4050 2500 50  0000 C CNN
-F 1 "CONN_01X02" V 4150 2350 50  0000 C CNN
-F 2 "Pin_Headers:Pin_Header_Straight_1x02" H 4050 2350 50  0001 C CNN
-F 3 "" H 4050 2350 50  0000 C CNN
+F 0 "P3" H 4050 2500 50 0000 C CNN
+F 1 "CONN_01X02" V 4150 2350 50 0000 C CNN
+F 2 "Pin_Headers:Pin_Header_Straight_1x02" H 4050 2350 50 0001 C CNN
+F 3 "" H 4050 2350 50 0000 C CNN
 	1    4050 2350
 	1    0    0    -1
 $EndComp
-Wire Wire Line
-	3850 2300 3700 2300
-Wire Wire Line
-	3700 2400 3850 2400
 $Comp
 L CONN_01X02 P2
 U 1 1 57FC278D
 P 1650 2350
-F 0 "P2" H 1650 2500 50  0000 C CNN
-F 1 "CONN_01X02" V 1750 2350 50  0000 C CNN
-F 2 "Pin_Headers:Pin_Header_Straight_1x02" H 1650 2350 50  0001 C CNN
-F 3 "" H 1650 2350 50  0000 C CNN
+F 0 "P2" H 1650 2500 50 0000 C CNN
+F 1 "CONN_01X02" V 1750 2350 50 0000 C CNN
+F 2 "Pin_Headers:Pin_Header_Straight_1x02" H 1650 2350 50 0001 C CNN
+F 3 "" H 1650 2350 50 0000 C CNN
 	1    1650 2350
 	-1   0    0    1
@@
 U 1 1 57FC2AD4
 P 2150 1500
-F 0 "C1" H 2160 1570 50  0000 L CNN
-F 1 "0.1uF" H 2160 1420 50  0000 L CNN
-F 2 "Capacitors_SMD:C_1206_HandSoldering" H 2150 1500 50  0001 C CNN
-F 3 "" H 2150 1500 50  0000 C CNN
+F 0 "C1" H 2160 1570 50 0000 L CNN
+F 1 "0.1uF" H 2160 1420 50 0000 L CNN
+F 2 "Capacitors_SMD:C_1206_HandSoldering" H 2150 1500 50 0001 C CNN
+F 3 "" H 2150 1500 50 0000 C CNN
 	1    2150 1500
 	1    0    0    -1
@@
 U 1 1 57FC2CA8
 P 1650 1350
-F 0 "P1" H 1650 1500 50  0000 C CNN
-F 1 "CONN_01X02" V 1750 1350 50  0000 C CNN
-F 2 "Pin_Headers:Pin_Header_Straight_1x02" H 1650 1350 50  0001 C CNN
-F 3 "" H 1650 1350 50  0000 C CNN
+F 0 "P1" H 1650 1500 50 0000 C CNN
+F 1 "CONN_01X02" V 1750 1350 50 0000 C CNN
+F 2 "Pin_Headers:Pin_Header_Straight_1x02" H 1650 1350 50 0001 C CNN
+F 3 "" H 1650 1350 50 0000 C CNN
 	1    1650 1350
 	-1   0    0    1
 $EndComp
-Wire Wire Line
-	1850 1300 2450 1300
-Wire Wire Line
-	2150 1300 2150 1400
 $Comp
 L C_Small C2
 U 1 1 57FC2EA8
 P 2450 1500
-F 0 "C2" H 2460 1570 50  0000 L CNN
-F 1 "1uF" H 2460 1420 50  0000 L CNN
-F 2 "Capacitors_SMD:C_1206_HandSoldering" H 2450 1500 50  0001 C CNN
-F 3 "" H 2450 1500 50  0000 C CNN
+F 0 "C2" H 2460 1570 50 0000 L CNN
+F 1 "1uF" H 2460 1420 50 0000 L CNN
+F 2 "Capacitors_SMD:C_1206_HandSoldering" H 2450 1500 50 0001 C CNN
+F 3 "" H 2450 1500 50 0000 C CNN
 	1    2450 1500
 	1    0    0    -1
@@
 U 1 1 57FC2F21
 P 1900 1750
-F 0 "#PWR03" H 1900 1500 50  0001 C CNN
-F 1 "GND" H 1900 1600 50  0000 C CNN
-F 2 "" H 1900 1750 50  0000 C CNN
-F 3 "" H 1900 1750 50  0000 C CNN
+F 0 "#PWR03" H 1900 1500 50 0001 C CNN
+F 1 "GND" H 1900 1600 50 0000 C CNN
+F 2 "" H 1900 1750 50 0000 C CNN
+F 3 "" H 1900 1750 50 0000 C CNN
 	1    1900 1750
 	1    0    0    -1
 $EndComp
-Wire Wire Line
-	1850 1400 1900 1400
-Wire Wire Line
-	1900 1400 1900 1750
 $Comp
 L VDD #PWR04
 U 1 1 57FC3033
 P 2450 1250
-F 0 "#PWR04" H 2450 1100 50  0001 C CNN
-F 1 "VDD" H 2450 1400 50  0000 C CNN
-F 2 "" H 2450 1250 50  0000 C CNN
-F 3 "" H 2450 1250 50  0000 C CNN
+F 0 "#PWR04" H 2450 1100 50 0001 C CNN
+F 1 "VDD" H 2450 1400 50 0000 C CNN
+F 2 "" H 2450 1250 50 0000 C CNN
+F 3 "" H 2450 1250 50 0000 C CNN
 	1    2450 1250
 	1    0    0    -1
 $EndComp
-Wire Wire Line
-	2450 1250 2450 1400
-Connection ~ 2150 1300
-Connection ~ 2450 1300
-Wire Wire Line
-	1900 1700 2450 1700
-Wire Wire Line
-	2450 1700 2450 1600
-Connection ~ 1900 1700
-Wire Wire Line
-	2150 1600 2150 1700
-Connection ~ 2150 1700
 Text Label 1900 2300 0    60   ~ 0
 i0
@@
 Text Label 3700 2400 0    60   ~ 0
 o1
+Wire Wire Line
+	3350 2600 3500 2600
+Wire Wire Line
+	3500 2600 3500 2700
+Wire Wire Line
+	2850 2900 2850 3000
+Wire Wire Line
+	2200 2950 3500 2950
+Wire Wire Line
+	3500 2950 3500 2900
+Wire Wire Line
+	2350 2600 2200 2600
+Wire Wire Line
+	2200 2600 2200 2700
+Wire Wire Line
+	2200 2900 2200 2950
+Wire Wire Line
+	2350 2300 2200 2300
+Wire Wire Line
+	2350 2400 2200 2400
+Wire Wire Line
+	2000 2300 1850 2300
+Wire Wire Line
+	2000 2400 1850 2400
+Wire Wire Line
+	2850 2050 2850 2100
+Wire Wire Line
+	3500 2300 3350 2300
+Wire Wire Line
+	3350 2400 3500 2400
+Wire Wire Line
+	3850 2300 3700 2300
+Wire Wire Line
+	3700 2400 3850 2400
+Wire Wire Line
+	1850 1300 2450 1300
+Wire Wire Line
+	2150 1300 2150 1400
+Wire Wire Line
+	1850 1400 1900 1400
+Wire Wire Line
+	1900 1400 1900 1750
+Wire Wire Line
+	2450 1250 2450 1400
+Wire Wire Line
+	1900 1700 2450 1700
+Wire Wire Line
+	2450 1700 2450 1600
+Wire Wire Line
+	2150 1600 2150 1700
+Connection ~ 2850 2950
+Connection ~ 2150 1300
+Connection ~ 2450 1300
+Connection ~ 1900 1700
+Connection ~ 2150 1700
 $EndSCHEMATC
