File: flipflop/74LVC1G79GW/74LVC1G79GW.sch (KiCad schematic (older format))
At the start: 21 parts, among them P1 CONN_01X02, P10 CONN_01X01, P11 CONN_01X01, P12 CONN_01X01, P13 CONN_01X01, P14 CONN_01X01, P2 CONN_01X02, P3 CONN_01X01, P4 CONN_01X01, P5 CONN_01X01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

Commit message: Re-export gerbers at 0.1mm default line width, update .schs with KiField, wget wavegen ICL 8083
Parts:
- U1, U2, U3, U4: Dist [1] Part # (none) -> 595-SN74LVC2G74DCUR; Dist [1] Source (none) -> http://www2.mouser.com/ProductDetail/Texas-Instruments/SN74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; Mfr (none) -> Texas; Mfr Part # (none) -> SN74LVC2G74DCUR
