File: fv1/fv1.kicad_pcb (KiCad board)
At the start: 2 copper layers, 0 parts

Commit message: Good start on small dsp
Parts:
- added U1: NCP1117ST33T3G_MountingTab, TO_SOT_Packages_SMD:SOT-223, F.Cu at (221.7, 75.6)
- added U2: FV1, Housings_SOIC:SOIC-28W_7.5x17.9mm_Pitch1.27mm, F.Cu at (239.7, 81.8)
Changed lines of the file:
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@@
     (links 0)
     (no_connects 0)
-    (area 149.333332 89.415 193.485715 99.085)
+    (area 209.9 70.8 245.880002 92.95)
     (thickness 1.6)
     (drawings 0)
     (tracks 0)
     (zones 0)
-    (modules 0)
-    (nets 1)
+    (modules 2)
+    (nets 33)
   )
   (page A4)
@@
   )
   (net 0 "")
+  (net 1 "Net-(U1-Pad4)")
+  (net 2 "Net-(U1-Pad2)")
+  (net 3 "Net-(U1-Pad3)")
+  (net 4 "Net-(U1-Pad1)")
+  (net 5 "Net-(U2-Pad1)")
+  (net 6 "Net-(U2-Pad2)")
+  (net 7 "Net-(U2-Pad3)")
+  (net 8 "Net-(U2-Pad4)")
+  (net 9 "Net-(U2-Pad5)")
+  (net 10 "Net-(U2-Pad6)")
+  (net 11 "Net-(U2-Pad7)")
+  (net 12 "Net-(U2-Pad8)")
+  (net 13 "Net-(U2-Pad9)")
+  (net 14 "Net-(U2-Pad10)")
+  (net 15 "Net-(U2-Pad11)")
+  (net 16 "Net-(U2-Pad12)")
+  (net 17 "Net-(U2-Pad13)")
+  (net 18 "Net-(U2-Pad14)")
+  (net 19 "Net-(U2-Pad15)")
+  (net 20 "Net-(U2-Pad16)")
+  (net 21 "Net-(U2-Pad17)")
+  (net 22 "Net-(U2-Pad18)")
+  (net 23 "Net-(U2-Pad19)")
+  (net 24 "Net-(U2-Pad20)")
+  (net 25 "Net-(U2-Pad21)")
+  (net 26 "Net-(U2-Pad22)")
+  (net 27 "Net-(U2-Pad23)")
+  (net 28 "Net-(U2-Pad24)")
+  (net 29 "Net-(U2-Pad25)")
+  (net 30 "Net-(U2-Pad26)")
+  (net 31 "Net-(U2-Pad27)")
+  (net 32 "Net-(U2-Pad28)")
   (net_class Default "This is the default net class."
     (clearance 0.2)
@@
     (uvia_dia 0.3)
     (uvia_drill 0.1)
+    (add_net "Net-(U1-Pad1)")
+    (add_net "Net-(U1-Pad2)")
+    (add_net "Net-(U1-Pad3)")
+    (add_net "Net-(U1-Pad4)")
+    (add_net "Net-(U2-Pad1)")
+    (add_net "Net-(U2-Pad10)")
+    (add_net "Net-(U2-Pad11)")
+    (add_net "Net-(U2-Pad12)")
+    (add_net "Net-(U2-Pad13)")
+    (add_net "Net-(U2-Pad14)")
+    (add_net "Net-(U2-Pad15)")
+    (add_net "Net-(U2-Pad16)")
+    (add_net "Net-(U2-Pad17)")
+    (add_net "Net-(U2-Pad18)")
+    (add_net "Net-(U2-Pad19)")
+    (add_net "Net-(U2-Pad2)")
+    (add_net "Net-(U2-Pad20)")
+    (add_net "Net-(U2-Pad21)")
+    (add_net "Net-(U2-Pad22)")
+    (add_net "Net-(U2-Pad23)")
+    (add_net "Net-(U2-Pad24)")
+    (add_net "Net-(U2-Pad25)")
+    (add_net "Net-(U2-Pad26)")
+    (add_net "Net-(U2-Pad27)")
+    (add_net "Net-(U2-Pad28)")
+    (add_net "Net-(U2-Pad3)")
+    (add_net "Net-(U2-Pad4)")
+    (add_net "Net-(U2-Pad5)")
+    (add_net "Net-(U2-Pad6)")
+    (add_net "Net-(U2-Pad7)")
+    (add_net "Net-(U2-Pad8)")
+    (add_net "Net-(U2-Pad9)")
+  )
+  (module TO_SOT_Packages_SMD:SOT-223 (layer F.Cu)
+    (at 221.719048 75.647001)
+    (descr "module CMS SOT223 4 pins")
+    (tags "CMS SOT")
+    (attr smd)
+    (fp_text reference U1 (at 0 -0.762) (layer F.SilkS)
+      (effects (font (size 1 1) (thickness 0.15)))
+    )
+    (fp_text value NCP1117ST33T3G_MountingTab (at 0 0.762) (layer F.Fab)
+      (effects (font (size 1 1) (thickness 0.15)))
+    )
+    (fp_line (start -3.556 1.524) (end -3.556 4.572) (layer F.SilkS) (width 0.15))
+    (fp_line (start -3.556 4.572) (end 3.556 4.572) (layer F.SilkS) (width 0.15))
+    (fp_line (start 3.556 4.572) (end 3.556 1.524) (layer F.SilkS) (width 0.15))
+    (fp_line (start -3.556 -1.524) (end -3.556 -2.286) (layer F.SilkS) (width 0.15))
+    (fp_line (start -3.556 -2.286) (end -2.032 -4.572) (layer F.SilkS) (width 0.15))
+    (fp_line (start -2.032 -4.572) (end 2.032 -4.572) (layer F.SilkS) (width 0.15))
+    (fp_line (start 2.032 -4.572) (end 3.556 -2.286) (layer F.SilkS) (width 0.15))
+    (fp_line (start 3.556 -2.286) (end 3.556 -1.524) (layer F.SilkS) (width 0.15))
+    (pad 4 smd rect (at 0 -3.302) (size 3.6576 2.032) (layers F.Cu F.Paste F.Mask)
+      (net 1 "Net-(U1-Pad4)"))
+    (pad 2 smd rect (at 0 3.302) (size 1.016 2.032) (layers F.Cu F.Paste F.Mask)
+      (net 2 "Net-(U1-Pad2)"))
+    (pad 3 smd rect (at 2.286 3.302) (size 1.016 2.032) (layers F.Cu F.Paste F.Mask)
+      (net 3 "Net-(U1-Pad3)"))
+    (pad 1 smd rect (at -2.286 3.302) (size 1.016 2.032) (layers F.Cu F.Paste F.Mask)
+      (net 4 "Net-(U1-Pad1)"))
+    (model TO_SOT_Packages_SMD.3dshapes/SOT-223.wrl
+      (at (xyz 0 0 0))
+      (scale (xyz 0.4 0.4 0.4))
+      (rotate (xyz 0 0 0))
+    )
+  )
+  (module Housings_SOIC:SOIC-28W_7.5x17.9mm_Pitch1.27mm (layer F.Cu)
+    (at 239.705001 81.825)
+    (descr "28-Lead Plastic Small Outline (SO) - Wide, 7.50 mm Body [SOIC] (see Microchip Packaging Specification 00000049BS.pdf)")
+    (tags "SOIC 1.27")
+    (attr smd)
+    (fp_text reference U2 (at 0 -10.05) (layer F.SilkS)
+      (effects (font (size 1 1) (thickness 0.15)))
+    )
+    (fp_text value FV1 (at 0 10.05) (layer F.Fab)
+      (effects (font (size 1 1) (thickness 0.15)))
+    )
+    (fp_line (start -2.75 -8.95) (end 3.75 -8.95) (layer F.Fab) (width 0.15))
+    (fp_line (start 3.75 -8.95) (end 3.75 8.95) (layer F.Fab) (width 0.15))
+    (fp_line (start 3.75 8.95) (end -3.75 8.95) (layer F.Fab) (width 0.15))
+    (fp_line (start -3.75 8.95) (end -3.75 -7.95) (layer F.Fab) (width 0.15))
+    (fp_line (start -3.75 -7.95) (end -2.75 -8.95) (layer F.Fab) (width 0.15))
+    (fp_line (start -5.95 -9.3) (end -5.95 9.3) (layer F.CrtYd) (width 0.05))
+    (fp_line (start 5.95 -9.3) (end 5.95 9.3) (layer F.CrtYd) (width 0.05))
+    (fp_line (start -5.95 -9.3) (end 5.95 -9.3) (layer F.CrtYd) (width 0.05))
+    (fp_line (start -5.95 9.3) (end 5.95 9.3) (layer F.CrtYd) (width 0.05))
+    (fp_line (start -3.875 -9.125) (end -3.875 -8.875) (layer F.SilkS) (width 0.15))
+    (fp_line (start 3.875 -9.125) (end 3.875 -8.78) (layer F.SilkS) (width 0.15))
+    (fp_line (start 3.875 9.125) (end 3.875 8.78) (layer F.SilkS) (width 0.15))
+    (fp_line (start -3.875 9.125) (end -3.875 8.78) (layer F.SilkS) (width 0.15))
+    (fp_line (start -3.875 -9.125) (end 3.875 -9.125) (layer F.SilkS) (width 0.15))
+    (fp_line (start -3.875 9.125) (end 3.875 9.125) (layer F.SilkS) (width 0.15))
+    (fp_line (start -3.875 -8.875) (end -5.7 -8.875) (layer F.SilkS) (width 0.15))
+    (pad 1 smd rect (at -4.7 -8.255) (size 2 0.6) (layers F.Cu F.Paste F.Mask)
+      (net 5 "Net-(U2-Pad1)"))
+    (pad 2 smd rect (at -4.7 -6.985) (size 2 0.6) (layers F.Cu F.Paste F.Mask)
+      (net 6 "Net-(U2-Pad2)"))
+    (pad 3 smd rect (at -4.7 -5.715) (size 2 0.6) (layers F.Cu F.Paste F.Mask)
+      (net 7 "Net-(U2-Pad3)"))
+    (pad 4 smd rect (at -4.7 -4.445) (size 2 0.6) (layers F.Cu F.Paste F.Mask)
+      (net 8 "Net-(U2-Pad4)"))
+    (pad 5 smd rect (at -4.7 -3.175) (size 2 0.6) (layers F.Cu F.Paste F.Mask)
+      (net 9 "Net-(U2-Pad5)"))
+    (pad 6 smd rect (at -4.7 -1.905) (size 2 0.6) (layers F.Cu F.Paste F.Mask)
+      (net 10 "Net-(U2-Pad6)"))
+    (pad 7 smd rect (at -4.7 -0.635) (size 2 0.6) (layers F.Cu F.Paste F.Mask)
+      (net 11 "Net-(U2-Pad7)"))
+    (pad 8 smd rect (at -4.7 0.635) (size 2 0.6) (layers F.Cu F.Paste F.Mask)
+      (net 12 "Net-(U2-Pad8)"))
+    (pad 9 smd rect (at -4.7 1.905) (size 2 0.6) (layers F.Cu F.Paste F.Mask)
+      (net 13 "Net-(U2-Pad9)"))
+    (pad 10 smd rect (at -4.7 3.175) (size 2 0.6) (layers F.Cu F.Paste F.Mask)
+      (net 14 "Net-(U2-Pad10)"))
+    (pad 11 smd rect (at -4.7 4.445) (size 2 0.6) (layers F.Cu F.Paste F.Mask)
+      (net 15 "Net-(U2-Pad11)"))
+    (pad 12 smd rect (at -4.7 5.715) (size 2 0.6) (layers F.Cu F.Paste F.Mask)
+      (net 16 "Net-(U2-Pad12)"))
+    (pad 13 smd rect (at -4.7 6.985) (size 2 0.6) (layers F.Cu F.Paste F.Mask)
+      (net 17 "Net-(U2-Pad13)"))
+    (pad 14 smd rect (at -4.7 8.255) (size 2 0.6) (layers F.Cu F.Paste F.Mask)
+      (net 18 "Net-(U2-Pad14)"))
+    (pad 15 smd rect (at 4.7 8.255) (size 2 0.6) (layers F.Cu F.Paste F.Mask)
+      (net 19 "Net-(U2-Pad15)"))
+    (pad 16 smd rect (at 4.7 6.985) (size 2 0.6) (layers F.Cu F.Paste F.Mask)
+      (net 20 "Net-(U2-Pad16)"))
+    (pad 17 smd rect (at 4.7 5.715) (size 2 0.6) (layers F.Cu F.Paste F.Mask)
+      (net 21 "Net-(U2-Pad17)"))
+    (pad 18 smd rect (at 4.7 4.445) (size 2 0.6) (layers F.Cu F.Paste F.Mask)
+      (net 22 "Net-(U2-Pad18)"))
+    (pad 19 smd rect (at 4.7 3.175) (size 2 0.6) (layers F.Cu F.Paste F.Mask)
+      (net 23 "Net-(U2-Pad19)"))
+    (pad 20 smd rect (at 4.7 1.905) (size 2 0.6) (layers F.Cu F.Paste F.Mask)
+      (net 24 "Net-(U2-Pad20)"))
+    (pad 21 smd rect (at 4.7 0.635) (size 2 0.6) (layers F.Cu F.Paste F.Mask)
+      (net 25 "Net-(U2-Pad21)"))
+    (pad 22 smd rect (at 4.7 -0.635) (size 2 0.6) (layers F.Cu F.Paste F.Mask)
+      (net 26 "Net-(U2-Pad22)"))
+    (pad 23 smd rect (at 4.7 -1.905) (size 2 0.6) (layers F.Cu F.Paste F.Mask)
+      (net 27 "Net-(U2-Pad23)"))
+    (pad 24 smd rect (at 4.7 -3.175) (size 2 0.6) (layers F.Cu F.Paste F.Mask)
+      (net 28 "Net-(U2-Pad24)"))
+    (pad 25 smd rect (at 4.7 -4.445) (size 2 0.6) (layers F.Cu F.Paste F.Mask)
+      (net 29 "Net-(U2-Pad25)"))
+    (pad 26 smd rect (at 4.7 -5.715) (size 2 0.6) (layers F.Cu F.Paste F.Mask)
+      (net 30 "Net-(U2-Pad26)"))
+    (pad 27 smd rect (at 4.7 -6.985) (size 2 0.6) (layers F.Cu F.Paste F.Mask)
+      (net 31 "Net-(U2-Pad27)"))
+    (pad 28 smd rect (at 4.7 -8.255) (size 2 0.6) (layers F.Cu F.Paste F.Mask)
+      (net 32 "Net-(U2-Pad28)"))
+    (model Housings_SOIC.3dshapes/SOIC-28_7.5x17.9mm_Pitch1.27mm.wrl
+      (at (xyz 0 0 0))
+      (scale (xyz 1 1 1))
+      (rotate (xyz 0 0 0))
+    )
   )
 )
