File: fv1/fv1.sch (KiCad schematic (older format))
At the start: 0 parts

Commit message: Good start on small dsp
Parts:
- added C? (x3): .1u, symbol C_Small
- added C?: 10u, symbol C_Small
- added C?: 15pF, symbol C_Small
- added C? (x4): 1nF CGO, Capacitors_SMD:C_0805, symbol C_Small
- added C? (x4): 1uF, Capacitors_SMD:c_elec_4x5.8, symbol CP1_Small
- added D?: Red, symbol LED_Small
- added P? (x2): CONN_01X02, symbol CONN_01X02
- added P?: CONN_01X08, symbol CONN_01X08
- added P?: CONN_01X03, symbol CONN_01X03
- added P? (x2): CONN_01X04, symbol CONN_01X04
- added R?: 10, symbol R_Small
- added R?: 470, symbol R_Small
- added R? (x4): 470, Resistors_SMD:R_0805, symbol R_Small
- added R? (x4): 30k, Resistors_SMD:R_0805, symbol R_Small
- added U1: NCP1117ST33T3G_MountingTab, TO_SOT_Packages_SMD:SOT-223, symbol NCP1117ST33T3G_MountingTab
- added U2: FV1, Housings_SOIC:SOIC-28W_7.5x17.9mm_Pitch1.27mm, symbol FV1
Connections:
- new net: C?.1, R?.1, U2.1 (LIN)
- new net: P?.2 (P2), U2.13 (T0)
- new net: C?.1, R?.1, U2.2 (RIN)
- new net: C?.2, R?.1, U2.26 (REFP)
- new net: C?.1, U2.27 (ROUT)
- new net: C?.1, U2.28 (LOUT)
- new net: C?.2, U2.3 (MID)
- new net: R?.2, U2.5 (CLIP)
- new net: C?.2, U2.6 (AVDD), U2.8 (DVDD)
- new net: C?.2, U2.9 (X2)
- new net: D?.1 (K), R?.1
- new net: C?.1, R?.2 (x2)
- new net: C?.2, P?.3 (P3), R?.2
- new net: C?.1, P?.3 (P3), R?.1
- new net: C?.2, P?.1 (P1), R?.2
- new net: C?.2, R?.2, R?.2 (x2)
- new net: C?.1, P?.1 (P1), R?.1
- new net +3V3: C?.1, D?.2 (A), P?.3 (P3), R?.2, U2.23 (DVDD)
- new net 3V3: P?.1 (P1), U1.2 (VO), U1.4 (VO)
- new net Flash ADC/r0: P?.1 (P1)
- new net Flash ADC/r1: P?.2 (P2)
- new net Flash ADC/r2: P?.3 (P3)
- new net Flash ADC/r3: P?.4 (P4)
- new net Flash ADC/r4: P?.5 (P5)
- new net Flash ADC/r5: P?.6 (P6)
- new net Flash ADC/r6: P?.7 (P7)
- new net Flash ADC/r7: P?.8 (P8)
- new net GND: C?.1, C?.1, C?.1, C?.1, C?.2, C?.2, C?.2, C?.2, C?.2, P?.1 (P1), P?.1 (P1), P?.2 (P2), P?.2 (P2), P?.2 (P2), P?.4 (P4), P?.4 (P4), R?.1, R?.1, R?.1, R?.1, U1.1 (GND), U2.11 (GND), U2.12 (T1), U2.19 (GND), U2.24 (GND), U2.25 (REFN), U2.4 (GND), U2.7 (GND)
- new net POT0: U2.20 (POT0)
- new net POT1: U2.21 (POT1)
- new net POT2: U2.22 (POT2)
- new net S0: U2.16 (S0)
- new net S1: U2.17 (S1)
- new net S2: U2.18 (S2)
- new net SCK: U2.14 (SCK)
- new net SDA: U2.15 (SDA)
- new net VIN: P?.2 (P2), U1.3 (VI)
- new net X1: U2.10 (X1)
Other:
- note added: "EXT: H"
- note added: "INT: L"
- note added: "place\nnear\npin"

Commit message: Trump is president
Parts:
- removed P? (x2): CONN_01X02, symbol CONN_01X02
- added C?: 0.01uF, symbol C_Small
- added P? (x2): CONN_01X04, symbol CONN_01X04
- added P?: CONN_01X01, symbol CONN_01X01
- added R? (x2): 0, symbol R_Small
- added R?: 7.5k, symbol R_Small
- added RV? (x5): POT, symbol POT
- added U?: 24LC32A, symbol 24LC32A
- added U?: LM555N, symbol LM555N
Connections:
- net +3V3: now also R?.2, RV?.3, RV?.3, RV?.3, U?.8 (VCC), U?.8 (VCC)
- net 3V3: now also P?.2 (P2), P?.4 (P4)
- net GND: now also C?.2, P?.1 (P1), P?.2 (P2), P?.3 (P3), P?.4 (P4), R?.1, RV?.1, RV?.1, RV?.1, U?.1 (A0), U?.1 (GND), U?.2 (A1), U?.3 (A2), U?.4 (VSS), U?.7 (WP)
- net POT0: now also RV?.2
- net POT1: now also RV?.2
- net POT2: now also RV?.2
- net SDA: now also U?.5 (SDA)
- net VIN: now also P?.1 (P1), P?.3 (P3)
- net X1: now also R?.1, U?.3 (Q)
- net RIN: now reaches C?.2, P?.3 (P3), R?.2
- net RFV1: now reaches C?.1, R?.1
- net RFV1: no longer P?.3 (P3)
- net LIN: now reaches C?.2, P?.1 (P1), R?.2
- net LFV1: now reaches C?.1, R?.1
- net LFV1: no longer P?.1 (P1)
- net SCK renamed SCL
- net SCL: now also U?.6 (SCL)
- new net: C?.1, RV?.2, U?.2 (TR), U?.6 (THR)
- new net: RV?.2, U?.5 (CV)
- new net: R?.1, RV?.1
- new net: R?.2, RV?.3 (x2)
- new net LOUT: P?.1 (P1)
- new net PROG: P?.1 (P1)
- new net ROUT: P?.3 (P3)
Other:
- moved on the sheet: C?, D?, P?, R?, U1, U2
